Commit message: updating stompy model after leg changes, added tran to calf, added extra joints for rviz, fixed double joint publishing

File: src/stompy_description/urdf/stompyleg_macro.urdf.xacro (robot description, xacro)
@@ -233,30 +233,40 @@
   </joint>
   <!-- transmission added for gazebo_ros_control, needed for every joint -->
-  <transmission name="body_to_${name}_tran">
+  <transmission name="${prefix}body_to_${name}_tran">
     <type>transmission_interface/SimpleTransmission</type>
     <joint name="${prefix}body_to_${name}">
       <hardwareInterface>EffortJointInterface</hardwareInterface>
     </joint>
-    <actuator name="body_to_${name}_motor">
-      <hardwareInterface>EffortJointInterface</hardwareInterface>
-      <mechanicalReduction>1</mechanicalReduction>
-    </actuator>
-  </transmission>
-  <transmission name="${name}_hip_to_thigh_tran">
+    <actuator name="${prefix}body_to_${name}_motor">
+      <hardwareInterface>EffortJointInterface</hardwareInterface>
+      <mechanicalReduction>1</mechanicalReduction>
+    </actuator>
+  </transmission>
+  <transmission name="${prefix}${name}_hip_to_thigh_tran">
     <type>transmission_interface/SimpleTransmission</type>
     <joint name="${prefix}${name}__hip_to_thigh">
       <hardwareInterface>EffortJointInterface</hardwareInterface>
     </joint>
-    <actuator name="${name}_hip_to_thigh_motor">
-      <hardwareInterface>EffortJointInterface</hardwareInterface>
-      <mechanicalReduction>1</mechanicalReduction>
-    </actuator>
-  </transmission>
-  <transmission name="${name}_thigh_to_calf_upper_tran">
+    <actuator name="${prefix}${name}_hip_to_thigh_motor">
+      <hardwareInterface>EffortJointInterface</hardwareInterface>
+      <mechanicalReduction>1</mechanicalReduction>
+    </actuator>
+  </transmission>
+  <transmission name="${prefix}${name}_thigh_to_calf_upper_tran">
     <type>transmission_interface/SimpleTransmission</type>
     <joint name="${prefix}${name}__thigh_to_calf_upper">
       <hardwareInterface>EffortJointInterface</hardwareInterface>
     </joint>
-    <actuator name="${name}_thigh_to_calf_upper_motor">
+    <actuator name="${prefix}${name}_thigh_to_calf_upper_motor">
+      <hardwareInterface>EffortJointInterface</hardwareInterface>
+      <mechanicalReduction>1</mechanicalReduction>
+    </actuator>
+  </transmission>
+  <transmission name="${prefix}${name}_calf_upper_to_calf_lower_tran">
+    <type>transmission_interface/SimpleTransmission</type>
+    <joint name="${prefix}${name}__calf_upper_to_calf_lower">
+      <hardwareInterface>EffortJointInterface</hardwareInterface>
+    </joint>
+    <actuator name="${prefix}${name}_calf_upper_to_calf_lower_motor">
       <hardwareInterface>EffortJointInterface</hardwareInterface>
       <mechanicalReduction>1</mechanicalReduction>

Commit message: stand and move work, effort, damping and pid tweaking
- large increase of max effort
- adding better shock
- adding initial srdf
- wip joint damping
- working on pids
- working on stand and move legs

File: src/stompy_description/urdf/stompyleg_macro.urdf.xacro (robot description, xacro)
@@ -1,5 +1,6 @@
 <?xml version="1.0" ?>
 <robot xmlns:xacro="http://www.ros.org/wiki/xacro">
- <xacro:property name="max_e" value="10000"/>
+ <xacro:property name="max_e" value="100000000000"/>
+ <!--<xacro:property name="max_e" value="1000000"/>-->
  <xacro:property name="max_v" value="10"/>
  <xacro:macro name="leg" params="prefix name rpy xyz">
@@ -9,5 +10,7 @@
     <origin rpy="0  0  0" xyz="0.279  0     0"/>
     <axis xyz="0  1  0"/>
-    <limit effort="${max_e}" lower="0.0" upper="0.6981" velocity="${max_v}"/>
+    <!--<limit effort="${max_e}" lower="0.0" upper="0.6981" velocity="${max_v}"/>-->
+    <limit effort="${max_e}" lower="0.0" upper="1.178" velocity="${max_v}"/>
+    <dynamics damping="10.0" />
   </joint>
   <joint name="${prefix}${name}__thigh_to_calf_upper" type="revolute">
@@ -16,5 +19,7 @@
     <origin rpy="0  0  0" xyz="0.14399  0       1.364"/>
     <axis xyz="0  1  0"/>
-    <limit effort="${max_e}" lower="-0.6981" upper="0.0" velocity="${max_v}"/>
+    <!--<limit effort="${max_e}" lower="-0.6981" upper="0.0" velocity="${max_v}"/>-->
+    <limit effort="${max_e}" lower="-1.178" upper="0.0" velocity="${max_v}"/>
+    <dynamics damping="10.0" />
   </joint>
   <joint name="${prefix}${name}__calf_upper_to_linkage_upper" type="fixed">
@@ -24,4 +29,5 @@
     <axis xyz="0  1  0"/>
     <limit effort="${max_e}" lower="0" upper="0" velocity="${max_v}"/>
+    <dynamics damping="10.0" />
   </joint>
   <joint name="${prefix}${name}__calf_upper_to_linkage_lower" type="fixed">
@@ -31,4 +37,5 @@
     <axis xyz="0  1  0"/>
     <limit effort="${max_e}" lower="0" upper="0" velocity="${max_v}"/>
+    <dynamics damping="10.0" />
   </joint>
   <joint name="${prefix}${name}__calf_upper_to_calf_lower" type="prismatic">
@@ -39,6 +46,8 @@
     <axis xyz="0  0  1"/>
     <!-- TODO sort out shock -->
-    <limit effort="${max_e}" lower="-0.0527" upper="0.0527" velocity="${max_v}"/>
+    <!--<limit effort="${max_e}" lower="-0.0527" upper="0.0527" velocity="${max_v}"/>-->
+    <limit effort="10942" lower="0.0" upper="0.104" velocity="${max_v}"/>
     <!--<limit effort="3000" lower="0.0" upper="0.0" velocity="${max_v}"/>-->
+    <dynamics damping="10.0" />
   </joint>
   <!--
@@ -64,4 +73,5 @@
     <axis xyz="0  1  0"/>
     <limit effort="${max_e}" lower="-1.3962" upper="1.3962" velocity="${max_v}"/>
+    <dynamics damping="10.0" />
   </joint>
   <joint name="${prefix}${name}__ankle_to_foot" type="revolute">
@@ -71,4 +81,5 @@
     <axis xyz="1  0  0"/>
     <limit effort="${max_e}" lower="-1.3962" upper="1.3962" velocity="${max_v}"/>
+    <dynamics damping="10.0" />
   </joint>
   <!-- TODO footpad -->
@@ -175,4 +186,5 @@
     </inertial>
     <collision name="${prefix}${name}__collision">
+      <!--TODO figure out if this position is with a compressed shock -->
       <origin rpy="0  0  0" xyz="0.01567  0      -0.10663"/>
       <geometry>
@@ -231,4 +243,5 @@
     <axis xyz="0  0  1"/>
     <limit effort="${max_e}" lower="-1.57079" upper="1.57079" velocity="${max_v}"/>
+    <dynamics damping="10.0" />
   </joint>
   <!-- transmission added for gazebo_ros_control, needed for every joint -->

Commit message: fixing joint limits

File: src/stompy_description/urdf/stompyleg_macro.urdf.xacro (robot description, xacro)
@@ -11,5 +11,5 @@
     <axis xyz="0  1  0"/>
     <!--<limit effort="${max_e}" lower="0.0" upper="0.6981" velocity="${max_v}"/>-->
-    <limit effort="${max_e}" lower="0.0" upper="1.178" velocity="${max_v}"/>
+    <limit effort="${max_e}" lower="0.0" upper="1.5708" velocity="${max_v}"/>
     <dynamics damping="10.0" />
   </joint>
@@ -20,5 +20,5 @@
     <axis xyz="0  1  0"/>
     <!--<limit effort="${max_e}" lower="-0.6981" upper="0.0" velocity="${max_v}"/>-->
-    <limit effort="${max_e}" lower="-1.178" upper="0.0" velocity="${max_v}"/>
+    <limit effort="${max_e}" lower="-2.3736" upper="0.0" velocity="${max_v}"/>
     <dynamics damping="10.0" />
   </joint>
@@ -242,5 +242,5 @@
     <origin rpy="${rpy}" xyz="${xyz}"/>
     <axis xyz="0  0  1"/>
-    <limit effort="${max_e}" lower="-1.57079" upper="1.57079" velocity="${max_v}"/>
+    <limit effort="${max_e}" lower="-1.178" upper="1.178" velocity="${max_v}"/>
     <dynamics damping="10.0" />
   </joint>

Commit message: switching back to effort control

File: src/stompy_description/urdf/stompyleg_macro.urdf.xacro (robot description, xacro)
@@ -79,4 +79,5 @@
     <dynamics damping="10.0" />
   </joint>
+  <!--
   <joint name="${prefix}${name}__foot_to_pad" type="continuous">
     <parent link="${prefix}${name}__foot"/>
@@ -84,9 +85,6 @@
     <origin rpy="0 0 0" xyz="0 0 -0.153"/>
     <axis xyz="0 0 1"/>
-    <!--
-    <limit effort="${max_e}" lower="0" upper="0" velocity="${max_v}"/>
-    <dynamics damping="1000.0" />
-    -->
-  </joint>
+  </joint>
+  -->
   <link name="${prefix}${name}__hip">
     <inertial>
@@ -243,4 +241,5 @@
     </visual>
   </link>
+  <!--
   <link name="${prefix}${name}__pad">
     <inertial>
@@ -263,10 +262,11 @@
   </link>
   <gazebo reference="${prefix}${name}__pad">
-    <mu1>15000000000</mu1>
-    <mu2>15000000000</mu2>
+    <mu1>50</mu1>
+    <mu2>50</mu2>
     <fdir1>0 0 0</fdir1>
     <minDepth>0.0001</minDepth>
-    <maxVel>100000.0</maxVel>
+    <maxVel>1000000000.0</maxVel>
   </gazebo>
+  -->
   <joint name="${prefix}body_to_${name}" type="revolute">
     <parent link="${prefix}body"/>

Commit message: position control working, still some physics bugs

File: src/stompy_description/urdf/stompyleg_macro.urdf.xacro (robot description, xacro)
@@ -1,5 +1,5 @@
 <?xml version="1.0" ?>
 <robot xmlns:xacro="http://www.ros.org/wiki/xacro">
- <xacro:property name="max_e" value="100000000000"/>
+ <xacro:property name="max_e" value="1000000"/>
  <xacro:property name="max_v" value="10"/>
  <xacro:macro name="leg" params="prefix name rpy xyz">

Commit message: push before switching from position control

File: src/stompy_description/urdf/stompyleg_macro.urdf.xacro (robot description, xacro)
@@ -78,5 +78,5 @@
     <limit effort="${max_e}" lower="-1.3962" upper="1.3962" velocity="${max_v}"/>
     <dynamics damping="10.0" />
-  </joint>
+</joint>
   <!--
   <joint name="${prefix}${name}__foot_to_pad" type="continuous">
@@ -240,5 +240,17 @@
       </geometry>
     </visual>
-  </link>
+</link>
+  <gazebo reference="${prefix}${name}__foot">
+    <mu1>100000000000</mu1>
+    <mu2>100000000000</mu2>
+    <!--
+    <fdir1>0 1 0</fdir1>
+    -->
+    <kp>100000000000000.0</kp>
+    <kd>0.00001</kd>
+    <minDepth>0.003</minDepth>
+  </gazebo>
+<!--
+  -->
   <!--
   <link name="${prefix}${name}__pad">

Commit message: effort based position control using high damping

File: src/stompy_description/urdf/stompyleg_macro.urdf.xacro (robot description, xacro)
@@ -1,5 +1,5 @@
 <?xml version="1.0" ?>
 <robot xmlns:xacro="http://www.ros.org/wiki/xacro">
- <xacro:property name="max_e" value="1000000"/>
+ <xacro:property name="max_e" value="10000000"/>
  <xacro:property name="max_v" value="10"/>
  <xacro:macro name="leg" params="prefix name rpy xyz">
@@ -10,5 +10,5 @@
     <axis xyz="0  1  0"/>
     <limit effort="${max_e}" lower="0.0" upper="1.5708" velocity="${max_v}"/>
-    <dynamics damping="10.0" />
+    <dynamics damping="10000.0" />
   </joint>
   <joint name="${prefix}${name}__thigh_to_calf_upper" type="revolute">
@@ -19,5 +19,5 @@
     <!--<limit effort="${max_e}" lower="-0.6981" upper="0.0" velocity="${max_v}"/>-->
     <limit effort="${max_e}" lower="-2.3736" upper="0.0" velocity="${max_v}"/>
-    <dynamics damping="10.0" />
+    <dynamics damping="10000.0" />
   </joint>
   <!--
@@ -28,5 +28,5 @@
     <axis xyz="0  1  0"/>
     <limit effort="${max_e}" lower="0" upper="0" velocity="${max_v}"/>
-    <dynamics damping="10.0" />
+    <dynamics damping="10000.0" />
   </joint>
   <joint name="${prefix}${name}__calf_upper_to_linkage_lower" type="fixed">
@@ -36,5 +36,5 @@
     <axis xyz="0  1  0"/>
     <limit effort="${max_e}" lower="0" upper="0" velocity="${max_v}"/>
-    <dynamics damping="10.0" />
+    <dynamics damping="10000.0" />
   </joint>
   -->
@@ -45,5 +45,5 @@
     <axis xyz="0  0  1"/>
     <limit effort="10942" lower="0.0" upper="0.104" velocity="${max_v}"/>
-    <dynamics damping="10.0" />
+    <dynamics damping="10000.0" />
   </joint>
   <!--
@@ -69,5 +69,5 @@
     <axis xyz="0  1  0"/>
     <limit effort="${max_e}" lower="-1.3962" upper="1.3962" velocity="${max_v}"/>
-    <dynamics damping="10.0" />
+    <dynamics damping="30.0" />
   </joint>
   <joint name="${prefix}${name}__ankle_to_foot" type="revolute">
@@ -77,5 +77,5 @@
     <axis xyz="1  0  0"/>
     <limit effort="${max_e}" lower="-1.3962" upper="1.3962" velocity="${max_v}"/>
-    <dynamics damping="10.0" />
+    <dynamics damping="30.0" />
 </joint>
   <!--
@@ -242,11 +242,6 @@
 </link>
   <gazebo reference="${prefix}${name}__foot">
-    <mu1>100000000000</mu1>
-    <mu2>100000000000</mu2>
-    <!--
-    <fdir1>0 1 0</fdir1>
-    -->
-    <kp>100000000000000.0</kp>
-    <kd>0.00001</kd>
+    <mu1>50</mu1>
+    <mu2>50</mu2>
     <minDepth>0.003</minDepth>
   </gazebo>
@@ -287,5 +282,5 @@
     <axis xyz="0  0  1"/>
     <limit effort="${max_e}" lower="-1.178" upper="1.178" velocity="${max_v}"/>
-    <dynamics damping="10.0" />
+    <dynamics damping="10000.0" />
   </joint>
   <!-- transmission added for gazebo_ros_control, needed for every joint -->
@@ -293,8 +288,8 @@
     <type>transmission_interface/SimpleTransmission</type>
     <joint name="${prefix}body_to_${name}">
-      <hardwareInterface>PositionJointInterface</hardwareInterface>
+      <hardwareInterface>EffortJointInterface</hardwareInterface>
     </joint>
     <actuator name="${prefix}body_to_${name}_motor">
-      <hardwareInterface>PositionJointInterface</hardwareInterface>
+      <hardwareInterface>EffortJointInterface</hardwareInterface>
       <mechanicalReduction>1</mechanicalReduction>
     </actuator>
@@ -303,8 +298,8 @@
     <type>transmission_interface/SimpleTransmission</type>
     <joint name="${prefix}${name}__hip_to_thigh">
-      <hardwareInterface>PositionJointInterface</hardwareInterface>
+      <hardwareInterface>EffortJointInterface</hardwareInterface>
     </joint>
     <actuator name="${prefix}${name}_hip_to_thigh_motor">
-      <hardwareInterface>PositionJointInterface</hardwareInterface>
+      <hardwareInterface>EffortJointInterface</hardwareInterface>
       <mechanicalReduction>1</mechanicalReduction>
     </actuator>
@@ -313,8 +308,8 @@
     <type>transmission_interface/SimpleTransmission</type>
     <joint name="${prefix}${name}__thigh_to_calf_upper">
-      <hardwareInterface>PositionJointInterface</hardwareInterface>
+      <hardwareInterface>EffortJointInterface</hardwareInterface>
     </joint>
     <actuator name="${prefix}${name}_thigh_to_calf_upper_motor">
-      <hardwareInterface>PositionJointInterface</hardwareInterface>
+      <hardwareInterface>EffortJointInterface</hardwareInterface>
       <mechanicalReduction>1</mechanicalReduction>
     </actuator>

Commit message: updates to stompy world and leg to improve simulation

File: src/stompy_description/urdf/stompyleg_macro.urdf.xacro (robot description, xacro)
@@ -69,5 +69,5 @@
     <axis xyz="0  1  0"/>
     <limit effort="${max_e}" lower="-1.3962" upper="1.3962" velocity="${max_v}"/>
-    <dynamics damping="30.0" />
+    <dynamics damping="1.0" />
   </joint>
   <joint name="${prefix}${name}__ankle_to_foot" type="revolute">
@@ -77,7 +77,6 @@
     <axis xyz="1  0  0"/>
     <limit effort="${max_e}" lower="-1.3962" upper="1.3962" velocity="${max_v}"/>
-    <dynamics damping="30.0" />
+    <dynamics damping="1.0" />
 </joint>
-  <!--
   <joint name="${prefix}${name}__foot_to_pad" type="continuous">
     <parent link="${prefix}${name}__foot"/>
@@ -86,5 +85,4 @@
     <axis xyz="0 0 1"/>
   </joint>
-  -->
   <link name="${prefix}${name}__hip">
     <inertial>
@@ -244,9 +242,7 @@
     <mu1>50</mu1>
     <mu2>50</mu2>
-    <minDepth>0.003</minDepth>
+    <maxVel>1000.0</maxVel>
+    <minDepth>0.0000003</minDepth>
   </gazebo>
-<!--
-  -->
-  <!--
   <link name="${prefix}${name}__pad">
     <inertial>
@@ -269,11 +265,9 @@
   </link>
   <gazebo reference="${prefix}${name}__pad">
-    <mu1>50</mu1>
-    <mu2>50</mu2>
-    <fdir1>0 0 0</fdir1>
-    <minDepth>0.0001</minDepth>
-    <maxVel>1000000000.0</maxVel>
+    <mu1>500</mu1>
+    <mu2>500</mu2>
+    <maxVel>1000.0</maxVel>
+    <minDepth>0.0000003</minDepth>
   </gazebo>
-  -->
   <joint name="${prefix}body_to_${name}" type="revolute">
     <parent link="${prefix}body"/>
