Commit message: making leg hopefully more modular

File: src/stompy_description/urdf/stompyleg.urdf.xacro (robot description, xacro)
@@ -1,41 +1,46 @@
 <?xml version="1.0" ?>
-<robot xmlns:xacro="http://www.ros.org/wiki/xacro" name="stompy">
+<robot xmlns:xacro="http://www.ros.org/wiki/xacro" name="stompyleg">
 <!--
      build 6 legs and a body
  -->
+ <gazebo>
+  <plugin name="gazebo_ros_control" filename="libgazebo_ros_control.so">
+    <robotNamespace>/stompyleg</robotNamespace>
+  </plugin>
+ </gazebo>
  <xacro:property name="max_e" value="1000"/>
  <xacro:property name="max_v" value="10"/>
- <xacro:macro name="leg" params="name rpy xyz">
-  <joint name="stompy__${name}__hip_to_thigh" type="revolute">
-    <parent link="stompy__${name}__hip"/>
-    <child link="stompy__${name}__thigh"/>
+ <xacro:macro name="leg" params="prefix name rpy xyz">
+  <joint name="${prefix}${name}__hip_to_thigh" type="revolute">
+    <parent link="${prefix}${name}__hip"/>
+    <child link="${prefix}${name}__thigh"/>
     <origin rpy="0  0  0" xyz="0.279  0     0"/>
     <axis xyz="0  1  0"/>
     <limit effort="${max_e}" lower="0.0" upper="0.6981" velocity="${max_v}"/>
   </joint>
-  <joint name="stompy__${name}__thigh_to_calf_upper" type="revolute">
-    <parent link="stompy__${name}__thigh"/>
-    <child link="stompy__${name}__calf_upper"/>
+  <joint name="${prefix}${name}__thigh_to_calf_upper" type="revolute">
+    <parent link="${prefix}${name}__thigh"/>
+    <child link="${prefix}${name}__calf_upper"/>
     <origin rpy="0  0  0" xyz="0.14399  0       1.364"/>
     <axis xyz="0  1  0"/>
     <limit effort="${max_e}" lower="-0.6981" upper="0.0" velocity="${max_v}"/>
   </joint>
-  <joint name="stompy__${name}__calf_upper_to_linkage_upper" type="fixed">
-    <parent link="stompy__${name}__calf_upper"/>
-    <child link="stompy__${name}__linkage_upper"/>
+  <joint name="${prefix}${name}__calf_upper_to_linkage_upper" type="fixed">
+    <parent link="${prefix}${name}__calf_upper"/>
+    <child link="${prefix}${name}__linkage_upper"/>
     <origin rpy="0  0  0" xyz="0.0016  0     -0.8185"/>
     <axis xyz="0  1  0"/>
     <limit effort="${max_e}" lower="0" upper="0" velocity="${max_v}"/>
   </joint>
-  <joint name="stompy__${name}__calf_upper_to_linkage_lower" type="fixed">
-    <parent link="stompy__${name}__calf_upper"/>
-    <child link="stompy__${name}__linkage_lower"/>
+  <joint name="${prefix}${name}__calf_upper_to_linkage_lower" type="fixed">
+    <parent link="${prefix}${name}__calf_upper"/>
+    <child link="${prefix}${name}__linkage_lower"/>
     <origin rpy="0  0  0" xyz="0.0388  0     -1.121"/>
     <axis xyz="0  1  0"/>
     <limit effort="${max_e}" lower="0" upper="0" velocity="${max_v}"/>
   </joint>
-  <joint name="stompy__${name}__calf_upper_to_calf_lower" type="prismatic">
-    <parent link="stompy__${name}__calf_upper"/>
-    <child link="stompy__${name}__calf_lower"/>
+  <joint name="${prefix}${name}__calf_upper_to_calf_lower" type="prismatic">
+    <parent link="${prefix}${name}__calf_upper"/>
+    <child link="${prefix}${name}__calf_lower"/>
     <!-- somewhat guesses... -->
     <origin rpy="0  0  0" xyz="0.2418  0   -1.121"/>
@@ -44,14 +49,14 @@
   </joint>
   <!--
-  <joint name="stompy__${name}__linkage_upper_to_calf_lower" type="revolute">
-    <parent link="stompy__${name}__linkage_upper"/>
-    <child link="stompy__${name}__calf_lower"/>
+  <joint name="${prefix}${name}__linkage_upper_to_calf_lower" type="revolute">
+    <parent link="${prefix}${name}__linkage_upper"/>
+    <child link="${prefix}${name}__calf_lower"/>
     <origin rpy="0  0  0" xyz="0.203  0     0"/>
     <axis xyz="0  1  0"/>
     <limit effort="${max_e}" lower="0.0" upper="0.349" velocity="${max_v}"/>
   </joint>
-  <joint name="stompy__${name}__linkage_lower_to_calf_lower" type="fixed">
-    <parent link="stompy__${name}__linkage_lower"/>
-    <child link="stompy__${name}__calf_lower"/>
+  <joint name="${prefix}${name}__linkage_lower_to_calf_lower" type="fixed">
+    <parent link="${prefix}${name}__linkage_lower"/>
+    <child link="${prefix}${name}__calf_lower"/>
     <origin rpy="0  0  0" xyz="2.02900000e-01   0.00000000e+00   1.00000000e-04"/>
     <axis xyz="0  1  0"/>
@@ -59,19 +64,19 @@
   </joint>
   -->
-  <joint name="stompy__${name}__calf_lower_to_ankle" type="revolute">
-    <parent link="stompy__${name}__calf_lower"/>
-    <child link="stompy__${name}__ankle"/>
+  <joint name="${prefix}${name}__calf_lower_to_ankle" type="revolute">
+    <parent link="${prefix}${name}__calf_lower"/>
+    <child link="${prefix}${name}__ankle"/>
     <origin rpy="0  0  0" xyz="-0.0171  0     -0.6656"/>
     <axis xyz="0  1  0"/>
     <limit effort="${max_e}" lower="-1.3962" upper="1.3962" velocity="${max_v}"/>
   </joint>
-  <joint name="stompy__${name}__ankle_to_foot" type="revolute">
-    <parent link="stompy__${name}__ankle"/>
-    <child link="stompy__${name}__foot"/>
+  <joint name="${prefix}${name}__ankle_to_foot" type="revolute">
+    <parent link="${prefix}${name}__ankle"/>
+    <child link="${prefix}${name}__foot"/>
     <origin rpy="0  0  0" xyz="0      0     -0.0412"/>
     <axis xyz="1  0  0"/>
     <limit effort="${max_e}" lower="-1.3962" upper="1.3962" velocity="${max_v}"/>
   </joint>
-  <link name="stompy__${name}__hip">
+  <link name="${prefix}${name}__hip">
     <inertial>
       <mass value="28.231"/>
@@ -79,5 +84,5 @@
       <inertia ixx="0.417" ixy="0." ixz="0.026" iyy="0.327" iyz="0." izz="0.337"/>
     </inertial>
-    <collision name="stompy__${name}__collision">
+    <collision name="${prefix}${name}__collision">
       <origin rpy="0  0  0" xyz="0.1106   0       0.04218"/>
       <geometry>
@@ -85,5 +90,5 @@
       </geometry>
     </collision>
-    <visual name="stompy__${name}__visual">
+    <visual name="${prefix}${name}__visual">
       <origin rpy="0  0  0" xyz="0  0  0"/>
       <geometry>
@@ -92,5 +97,5 @@
     </visual>
   </link>
-  <link name="stompy__${name}__thigh">
+  <link name="${prefix}${name}__thigh">
     <inertial>
       <mass value="64.053"/>
@@ -98,5 +103,5 @@
       <inertia ixx="10.62" ixy="0." ixz="-0.34" iyy="10.92" iyz="0." izz="1.334"/>
     </inertial>
-    <collision name="stompy__${name}__collision">
+    <collision name="${prefix}${name}__collision">
       <origin rpy="0  0  0" xyz="-0.04764  0       0.70869"/>
       <geometry>
@@ -104,5 +109,5 @@
       </geometry>
     </collision>
-    <visual name="stompy__${name}__visual">
+    <visual name="${prefix}${name}__visual">
       <origin rpy="0  0  0" xyz="0  0  0"/>
       <geometry>
@@ -111,5 +116,5 @@
     </visual>
   </link>
-  <link name="stompy__${name}__calf_upper">
+  <link name="${prefix}${name}__calf_upper">
     <inertial>
       <mass value="39.145"/>
@@ -117,5 +122,5 @@
       <inertia ixx="5.471" ixy="0." ixz="1.148" iyy="5.636" iyz="0." izz="0.775"/>
     </inertial>
-    <collision name="stompy__${name}__collision">
+    <collision name="${prefix}${name}__collision">
       <origin rpy="0  0  0" xyz="3.28400000e-02  -1.00000000e-05  -3.32310000e-01"/>
       <geometry>
@@ -123,5 +128,5 @@
       </geometry>
     </collision>
-    <visual name="stompy__${name}__visual">
+    <visual name="${prefix}${name}__visual">
       <origin rpy="0  0  0" xyz="0  0  0"/>
       <geometry>
@@ -130,5 +135,5 @@
     </visual>
   </link>
-  <link name="stompy__${name}__linkage_upper">
+  <link name="${prefix}${name}__linkage_upper">
     <inertial>
       <mass value="3.754"/>
@@ -136,5 +141,5 @@
       <inertia ixx="0.028" ixy="0." ixz="0." iyy="0.022" iyz="0" izz="0.009"/>
     </inertial>
-    <collision name="stompy__${name}__collision">
+    <collision name="${prefix}${name}__collision">
       <origin rpy="0  0  0" xyz="1.01380000e-01   0.00000000e+00  -1.00000000e-05"/>
       <geometry>
@@ -142,5 +147,5 @@
       </geometry>
     </collision>
-    <visual name="stompy__${name}__visual">
+    <visual name="${prefix}${name}__visual">
       <origin rpy="0  0  0" xyz="0  0  0"/>
       <geometry>
@@ -149,5 +154,5 @@
     </visual>
   </link>
-  <link name="stompy__${name}__linkage_lower">
+  <link name="${prefix}${name}__linkage_lower">
     <inertial>
       <mass value="3.754"/>
@@ -155,5 +160,5 @@
       <inertia ixx="0.028" ixy="0." ixz="0." iyy="0.022" iyz="0" izz="0.009"/>
     </inertial>
-    <collision name="stompy__${name}__collision">
+    <collision name="${prefix}${name}__collision">
       <origin rpy="0  0  0" xyz="1.01380000e-01   0.00000000e+00  -1.00000000e-05"/>
       <geometry>
@@ -161,5 +166,5 @@
       </geometry>
     </collision>
-    <visual name="stompy__${name}__visual">
+    <visual name="${prefix}${name}__visual">
       <origin rpy="0  0  0" xyz="0  0  0"/>
       <geometry>
@@ -168,5 +173,5 @@
     </visual>
   </link>
-  <link name="stompy__${name}__calf_lower">
+  <link name="${prefix}${name}__calf_lower">
     <inertial>
       <mass value="18.983"/>
@@ -174,5 +179,5 @@
       <inertia ixx="1.827" ixy="0." ixz="0.243" iyy="1.859" iyz="0." izz="0.145"/>
     </inertial>
-    <collision name="stompy__${name}__collision">
+    <collision name="${prefix}${name}__collision">
       <origin rpy="0  0  0" xyz="0.01567  0      -0.10663"/>
       <geometry>
@@ -180,5 +185,5 @@
       </geometry>
     </collision>
-    <visual name="stompy__${name}__visual">
+    <visual name="${prefix}${name}__visual">
       <origin rpy="0  0  0" xyz="-0.0371  0      0.3024"/>
       <geometry>
@@ -187,5 +192,5 @@
     </visual>
   </link>
-  <link name="stompy__${name}__ankle">
+  <link name="${prefix}${name}__ankle">
     <inertial>
       <mass value="1.391"/>
@@ -193,5 +198,5 @@
       <inertia ixx="0.002" ixy="0" ixz="0" iyy="0.001" iyz="0" izz="0.002"/>
     </inertial>
-    <collision name="stompy__${name}__collision">
+    <collision name="${prefix}${name}__collision">
       <origin rpy="0  0  0" xyz="0       0      -0.01709"/>
       <geometry>
@@ -199,5 +204,5 @@
       </geometry>
     </collision>
-    <visual name="stompy__${name}__visual">
+    <visual name="${prefix}${name}__visual">
       <origin rpy="0  0  0" xyz="0  0  0"/>
       <geometry>
@@ -206,5 +211,5 @@
     </visual>
   </link>
-  <link name="stompy__${name}__foot">
+  <link name="${prefix}${name}__foot">
     <inertial>
       <mass value="9.307"/>
@@ -212,5 +217,5 @@
       <inertia ixx="0.069" ixy="0" ixz="0" iyy="0.069" iyz="0" izz="0.102"/>
     </inertial>
-    <collision name="stompy__${name}__collision">
+    <collision name="${prefix}${name}__collision">
       <origin rpy="0  0  0" xyz="0       0      -0.11187"/>
       <geometry>
@@ -218,5 +223,5 @@
       </geometry>
     </collision>
-    <visual name="stompy__${name}__visual">
+    <visual name="${prefix}${name}__visual">
       <origin rpy="0  0  0" xyz="0  0  0"/>
       <geometry>
@@ -225,13 +230,44 @@
     </visual>
   </link>
-  <joint name="stompy__body_to_${name}" type="revolute">
-    <parent link="stompy__body"/>
-    <child link="stompy__${name}__hip"/>
+  <joint name="${prefix}body_to_${name}" type="revolute">
+    <parent link="${prefix}body"/>
+    <child link="${prefix}${name}__hip"/>
     <origin rpy="${rpy}" xyz="${xyz}"/>
     <axis xyz="0  0  1"/>
     <limit effort="${max_e}" lower="-1.57079" upper="1.57079" velocity="${max_v}"/>
   </joint>
+  <!-- transmission added for gazebo_ros_control, needed for every joint -->
+  <transmission name="body_to_${name}_tran">
+    <type>transmission_interface/SimpleTransmission</type>
+    <joint name="${prefix}body_to_${name}">
+      <hardwareInterface>EffortJointInterface</hardwareInterface>
+    </joint>
+    <actuator name="body_to_${name}_motor">
+      <hardwareInterface>EffortJointInterface</hardwareInterface>
+      <mechanicalReduction>1</mechanicalReduction>
+    </actuator>
+  </transmission>
+  <transmission name="${name}_hip_to_thigh_tran">
+    <type>transmission_interface/SimpleTransmission</type>
+    <joint name="${prefix}${name}__hip_to_thigh">
+      <hardwareInterface>EffortJointInterface</hardwareInterface>
+    </joint>
+    <actuator name="${name}_hip_to_thigh_motor">
+      <hardwareInterface>EffortJointInterface</hardwareInterface>
+      <mechanicalReduction>1</mechanicalReduction>
+    </actuator>
+  </transmission>
+  <transmission name="${name}_thigh_to_calf_upper_tran">
+    <type>transmission_interface/SimpleTransmission</type>
+    <joint name="${prefix}${name}__thigh_to_calf_upper">
+      <hardwareInterface>EffortJointInterface</hardwareInterface>
+    </joint>
+    <actuator name="${name}_thigh_to_calf_upper_motor">
+      <hardwareInterface>EffortJointInterface</hardwareInterface>
+      <mechanicalReduction>1</mechanicalReduction>
+    </actuator>
+  </transmission>
  </xacro:macro>
- <link name="stompy__body">
+ <link name="stompyleg__body">
     <inertial>
       <mass value="1823.41"/>
@@ -240,5 +276,5 @@
       <inertia ixx="499.7" ixy="0.019" ixz="-172.0" iyy="3253.0" iyz="0.019" izz="3049.0"/>
     </inertial>
-    <collision name="stompy__collision">
+    <collision name="stompyleg__collision">
       <!--<origin rpy="0  0  0" xyz="0     0     1.495"/>-->
       <origin rpy="0  0  0" xyz="0     0     0.7"/>
@@ -247,5 +283,5 @@
       </geometry>
     </collision>
-    <visual name="stompy__visual">
+    <visual name="stompyleg__visual">
       <origin rpy="0  0  0" xyz="0  0  1"/>
       <geometry>
@@ -257,5 +293,5 @@
     </visual>
   </link>
-  <xacro:leg name="fl" rpy="0 0 0.7853" xyz="2.35117  0.5842   1.2"/>
+  <xacro:leg prefix="stompyleg__" name="fl" rpy="0 0 0.7853" xyz="2.35117  0.5842   1.2"/>
   <!--
   <xacro:leg name="fr" rpy="0      0     -0.7853" xyz="2.35117 -0.5842   1"/>

Commit message: fixing visual and physical stompyleg body

File: src/stompy_description/urdf/stompyleg.urdf.xacro (robot description, xacro)
@@ -284,5 +284,5 @@
     </collision>
     <visual name="stompyleg__visual">
-      <origin rpy="0  0  0" xyz="0  0  1"/>
+      <origin rpy="0  0  0" xyz="0  0  0.7"/>
       <geometry>
         <box size="4.47037 1.3716 1."/>

Commit message: fixing joint lengths, upping pid params

File: src/stompy_description/urdf/stompyleg.urdf.xacro (robot description, xacro)
@@ -40,6 +40,7 @@
     </visual>
   </link>
+  <xacro:leg prefix="stompyleg__" name="fl" rpy="0 0 0" xyz="2.35117  0.5842   1.2"/>
+  <!--
   <xacro:leg prefix="stompyleg__" name="fl" rpy="0 0 0.7853" xyz="2.35117  0.5842   1.2"/>
-  <!--
   <xacro:leg name="fr" rpy="0      0     -0.7853" xyz="2.35117 -0.5842   1"/>
   <xacro:leg name="ml" rpy="0      0      1.5706" xyz="0.11597  0.6858   1"/>

File: src/stompy_description/urdf/stompyleg_macro.urdf.xacro (robot description, xacro)
@@ -8,5 +8,5 @@
     <parent link="${prefix}${name}__hip"/>
     <child link="${prefix}${name}__thigh"/>
-    <origin rpy="0  0  0" xyz="0.279  0     0"/>
+    <origin rpy="0  0  0" xyz="0.2794  0     0"/>
     <axis xyz="0  1  0"/>
     <!--<limit effort="${max_e}" lower="0.0" upper="0.6981" velocity="${max_v}"/>-->
@@ -17,5 +17,5 @@
     <parent link="${prefix}${name}__thigh"/>
     <child link="${prefix}${name}__calf_upper"/>
-    <origin rpy="0  0  0" xyz="0.14399  0       1.364"/>
+    <origin rpy="0  0  0" xyz="0.144  0       1.36402"/>
     <axis xyz="0  1  0"/>
     <!--<limit effort="${max_e}" lower="-0.6981" upper="0.0" velocity="${max_v}"/>-->
@@ -43,5 +43,6 @@
     <child link="${prefix}${name}__calf_lower"/>
     <!-- somewhat guesses... -->
-    <origin rpy="0  0  0" xyz="0.2418  0   -1.121"/>
+    <!--<origin rpy="0  0  0" xyz="0.2418  0   -1.121"/>-->
+    <origin rpy="0  0  0" xyz="0.2418  0   -1.14935"/>
     <axis xyz="0  0  1"/>
     <!-- TODO sort out shock -->

Commit message: renaming stompyleg namespace to stompy

File: src/stompy_description/urdf/stompyleg.urdf.xacro (robot description, xacro)
@@ -1,4 +1,4 @@
 <?xml version="1.0" ?>
-<robot xmlns:xacro="http://www.ros.org/wiki/xacro" name="stompyleg">
+<robot xmlns:xacro="http://www.ros.org/wiki/xacro" name="stompy">
 <!--
      build 1 leg and a fake body
@@ -6,15 +6,15 @@
  <gazebo>
   <plugin name="gazebo_ros_control" filename="libgazebo_ros_control.so">
-    <robotNamespace>/stompyleg</robotNamespace>
+    <robotNamespace>/stompy</robotNamespace>
   </plugin>
  </gazebo>
  <xacro:include filename="$(find stompy_description)/urdf/stompyleg_macro.urdf.xacro" />
- <link name="stompyleg__base" />
- <joint name="stompyleg__base_to_body" type="fixed">
+ <link name="stompy__base" />
+ <joint name="stompy__base_to_body" type="fixed">
   <origin xyz="0 0 0" rpy="0 0 0"/>
-  <parent link="stompyleg__base" />
-  <child link="stompyleg__body" />
+  <parent link="stompy__base" />
+  <child link="stompy__body" />
  </joint>
- <link name="stompyleg__body">
+ <link name="stompy__body">
     <inertial>
       <mass value="1823.41"/>
@@ -23,5 +23,5 @@
       <inertia ixx="499.7" ixy="0.019" ixz="-172.0" iyy="3253.0" iyz="0.019" izz="3049.0"/>
     </inertial>
-    <collision name="stompyleg__collision">
+    <collision name="stompy__collision">
       <!--<origin rpy="0  0  0" xyz="0     0     1.495"/>-->
       <origin rpy="0  0  0" xyz="0     0     0.7"/>
@@ -30,5 +30,5 @@
       </geometry>
     </collision>
-    <visual name="stompyleg__visual">
+    <visual name="stompy__visual">
       <origin rpy="0  0  0" xyz="0  0  0.7"/>
       <geometry>
@@ -40,7 +40,7 @@
     </visual>
   </link>
-  <xacro:leg prefix="stompyleg__" name="fl" rpy="0 0 0" xyz="2.35117  0.5842   1.2"/>
+  <xacro:leg prefix="stompy__" name="fl" rpy="0 0 0" xyz="2.35117  0.5842   1.2"/>
   <!--
-  <xacro:leg prefix="stompyleg__" name="fl" rpy="0 0 0.7853" xyz="2.35117  0.5842   1.2"/>
+  <xacro:leg prefix="stompy__" name="fl" rpy="0 0 0.7853" xyz="2.35117  0.5842   1.2"/>
   <xacro:leg name="fr" rpy="0      0     -0.7853" xyz="2.35117 -0.5842   1"/>
   <xacro:leg name="ml" rpy="0      0      1.5706" xyz="0.11597  0.6858   1"/>
