Commit message: more updates to xacro and stand

File: src/stompy_description/urdf/stompy.urdf.xacro (robot description, xacro)
@@ -7,4 +7,10 @@
  </gazebo>
  <xacro:include filename="$(find stompy_description)/urdf/stompyleg_macro.urdf.xacro" />
+ <link name="stompy__base" />
+ <joint name="stompy__base_to_body" type="fixed">
+  <origin xyz="0 0 0" rpy="0 0 0"/>
+  <parent link="stompy__base" />
+  <child link="stompy__body" />
+ </joint>
  <link name="stompy__body">
     <inertial>

File: src/stompy_description/urdf/stompyleg.urdf.xacro (robot description, xacro)
@@ -10,4 +10,10 @@
  </gazebo>
  <xacro:include filename="$(find stompy_description)/urdf/stompyleg_macro.urdf.xacro" />
+ <link name="stompyleg__base" />
+ <joint name="stompyleg__base_to_body" type="fixed">
+  <origin xyz="0 0 0" rpy="0 0 0"/>
+  <parent link="stompyleg__base" />
+  <child link="stompyleg__body" />
+ </joint>
  <link name="stompyleg__body">
     <inertial>

File: src/stompy_description/urdf/stompyleg_macro.urdf.xacro (robot description, xacro)
@@ -38,5 +38,7 @@
     <origin rpy="0  0  0" xyz="0.2418  0   -1.121"/>
     <axis xyz="0  0  1"/>
+    <!-- TODO sort out shock -->
     <limit effort="${max_e}" lower="-0.0527" upper="0.0527" velocity="${max_v}"/>
+    <!--<limit effort="3000" lower="0.0" upper="0.0" velocity="${max_v}"/>-->
   </joint>
   <!--
@@ -70,4 +72,5 @@
     <limit effort="${max_e}" lower="-1.3962" upper="1.3962" velocity="${max_v}"/>
   </joint>
+  <!-- TODO footpad -->
   <link name="${prefix}${name}__hip">
     <inertial>

Commit message: updating before switch to velocity control

File: src/stompy_description/urdf/stompy.urdf.xacro (robot description, xacro)
@@ -16,15 +16,16 @@
     <inertial>
       <mass value="1823.41"/>
-      <origin rpy="0  0  0" xyz="0     0     1.495"/>
+      <!--<origin rpy="0  0  0" xyz="0     0     1.495"/>-->
+      <origin rpy="0  0  0" xyz="0     0     0"/>
       <inertia ixx="499.7" ixy="0.019" ixz="-172.0" iyy="3253.0" iyz="0.019" izz="3049.0"/>
     </inertial>
     <collision name="stompy__collision">
-      <origin rpy="0  0  0" xyz="0     0     1.495"/>
+      <origin rpy="0  0  0" xyz="0     0     0"/>
       <geometry>
-        <box size="4.47037 1.3716 1."/>
+        <box size="4.478688 1.168400 0.304800"/>
       </geometry>
     </collision>
     <visual name="stompy__visual">
-      <origin rpy="0  0  0" xyz="0  0  1"/>
+      <origin rpy="0  0  0" xyz="0  0  0"/>
       <geometry>
         <mesh filename="package://stompy_description/meshes/body.stl" scale="1.0 1.0 1.0"/>
@@ -32,9 +33,9 @@
     </visual>
   </link>
-  <xacro:leg prefix="stompy__" name="fl" rpy="0 0 0.7853" xyz="2.35117  0.5842   1"/>
-  <xacro:leg prefix="stompy__" name="fr" rpy="0      0     -0.7853" xyz="2.35117 -0.5842   1"/>
-  <xacro:leg prefix="stompy__" name="ml" rpy="0      0      1.5706" xyz="0.11597  0.6858   1"/>
-  <xacro:leg prefix="stompy__" name="mr" rpy="0      0     -1.5706" xyz="0.11597 -0.6858   1"/>
-  <xacro:leg prefix="stompy__" name="rl" rpy="0      0      2.3561" xyz="-2.1192  0.5842  1"/>
-  <xacro:leg prefix="stompy__" name="rr" rpy="0      0     -2.3561" xyz="-2.1192 -0.5842  1"/>
+  <xacro:leg prefix="stompy__" name="fl" rpy="0 0 0.7853" xyz="2.35117  0.5842   -0.0967"/>
+  <xacro:leg prefix="stompy__" name="fr" rpy="0      0     -0.7853" xyz="2.35117 -0.5842   -0.0967"/>
+  <xacro:leg prefix="stompy__" name="ml" rpy="0      0      1.5706" xyz="0.11597  0.6858   -0.0967"/>
+  <xacro:leg prefix="stompy__" name="mr" rpy="0      0     -1.5706" xyz="0.11597 -0.6858   -0.0967"/>
+  <xacro:leg prefix="stompy__" name="rl" rpy="0      0      2.3561" xyz="-2.1192  0.5842  -0.0967"/>
+  <xacro:leg prefix="stompy__" name="rr" rpy="0      0     -2.3561" xyz="-2.1192 -0.5842  -0.0967"/>
 </robot>

File: src/stompy_description/urdf/stompyleg_macro.urdf.xacro (robot description, xacro)
@@ -2,5 +2,4 @@
 <robot xmlns:xacro="http://www.ros.org/wiki/xacro">
  <xacro:property name="max_e" value="100000000000"/>
- <!--<xacro:property name="max_e" value="1000000"/>-->
  <xacro:property name="max_v" value="10"/>
  <xacro:macro name="leg" params="prefix name rpy xyz">
@@ -8,7 +7,6 @@
     <parent link="${prefix}${name}__hip"/>
     <child link="${prefix}${name}__thigh"/>
-    <origin rpy="0  0  0" xyz="0.2794  0     0"/>
-    <axis xyz="0  1  0"/>
-    <!--<limit effort="${max_e}" lower="0.0" upper="0.6981" velocity="${max_v}"/>-->
+    <origin rpy="0  0  0" xyz="0.279  0     0"/>
+    <axis xyz="0  1  0"/>
     <limit effort="${max_e}" lower="0.0" upper="1.5708" velocity="${max_v}"/>
     <dynamics damping="10.0" />
@@ -17,5 +15,5 @@
     <parent link="${prefix}${name}__thigh"/>
     <child link="${prefix}${name}__calf_upper"/>
-    <origin rpy="0  0  0" xyz="0.144  0       1.36402"/>
+    <origin rpy="0  0  0" xyz="0.143  0       1.364"/>
     <axis xyz="0  1  0"/>
     <!--<limit effort="${max_e}" lower="-0.6981" upper="0.0" velocity="${max_v}"/>-->
@@ -44,12 +42,7 @@
     <parent link="${prefix}${name}__calf_upper"/>
     <child link="${prefix}${name}__calf_lower"/>
-    <!-- somewhat guesses... -->
-    <!--<origin rpy="0  0  0" xyz="0.2418  0   -1.121"/>-->
-    <origin rpy="0  0  0" xyz="0.2418  0   -1.14935"/>
+    <origin rpy="0  0  0" xyz="0.203  0   -0.847"/>
     <axis xyz="0  0  1"/>
-    <!-- TODO sort out shock -->
-    <!--<limit effort="${max_e}" lower="-0.0527" upper="0.0527" velocity="${max_v}"/>-->
     <limit effort="10942" lower="0.0" upper="0.104" velocity="${max_v}"/>
-    <!--<limit effort="3000" lower="0.0" upper="0.0" velocity="${max_v}"/>-->
     <dynamics damping="10.0" />
   </joint>
@@ -73,5 +66,5 @@
     <parent link="${prefix}${name}__calf_lower"/>
     <child link="${prefix}${name}__ankle"/>
-    <origin rpy="0  0  0" xyz="-0.0171  0     -0.6656"/>
+    <origin rpy="0  0  0" xyz="0.02  0     -0.968"/>
     <axis xyz="0  1  0"/>
     <limit effort="${max_e}" lower="-1.3962" upper="1.3962" velocity="${max_v}"/>
@@ -86,18 +79,27 @@
     <dynamics damping="10.0" />
   </joint>
-  <!-- TODO footpad -->
+  <joint name="${prefix}${name}__foot_to_pad" type="continuous">
+    <parent link="${prefix}${name}__foot"/>
+    <child link="${prefix}${name}__pad"/>
+    <origin rpy="0 0 0" xyz="0 0 -0.153"/>
+    <axis xyz="0 0 1"/>
+    <!--
+    <limit effort="${max_e}" lower="0" upper="0" velocity="${max_v}"/>
+    <dynamics damping="1000.0" />
+    -->
+  </joint>
   <link name="${prefix}${name}__hip">
     <inertial>
       <mass value="28.231"/>
-      <origin rpy="0  0  0" xyz="0.11386  0       0.03317"/>
+      <origin rpy="0  0  0" xyz="0.114006 0.000000 0.032923"/>
       <inertia ixx="0.417" ixy="0." ixz="0.026" iyy="0.327" iyz="0." izz="0.337"/>
     </inertial>
-    <collision name="${prefix}${name}__collision">
-      <origin rpy="0  0  0" xyz="0.1106   0       0.04218"/>
+    <collision name="${prefix}${name}__hip_collision">
+      <origin rpy="0  0  0" xyz="0.1341685 -0.000000 0.096707"/>
       <geometry>
         <box size="0.388937 0.411136 0.304614"/>
       </geometry>
     </collision>
-    <visual name="${prefix}${name}__visual">
+    <visual name="${prefix}${name}__hip_visual">
       <origin rpy="0  0  0" xyz="0  0  0"/>
       <geometry>
@@ -109,14 +111,14 @@
     <inertial>
       <mass value="64.053"/>
-      <origin rpy="0  0  0" xyz="-0.04116  0       0.52666"/>
+      <origin rpy="0  0  0" xyz="-0.041591 -0.000000 0.526720"/>
       <inertia ixx="10.62" ixy="0." ixz="-0.34" iyy="10.92" iyz="0." izz="1.334"/>
     </inertial>
-    <collision name="${prefix}${name}__collision">
-      <origin rpy="0  0  0" xyz="-0.04764  0       0.70869"/>
+    <collision name="${prefix}${name}__thigh_collision">
+      <origin rpy="0  0  0" xyz="-0.078093 -0.000000 0.6820835"/>
       <geometry>
         <box size="0.525414 0.273050 1.446567"/>
       </geometry>
     </collision>
-    <visual name="${prefix}${name}__visual">
+    <visual name="${prefix}${name}__thigh_visual">
       <origin rpy="0  0  0" xyz="0  0  0"/>
       <geometry>
@@ -128,14 +130,14 @@
     <inertial>
       <mass value="39.145"/>
-      <origin rpy="0  0  0" xyz="0.03528  0      -0.33951"/>
+      <origin rpy="0  0  0" xyz="0.035211 -0.000003 -0.339598"/>
       <inertia ixx="5.471" ixy="0." ixz="1.148" iyy="5.636" iyz="0." izz="0.775"/>
     </inertial>
-    <collision name="${prefix}${name}__collision">
-      <origin rpy="0  0  0" xyz="3.28400000e-02  -1.00000000e-05  -3.32310000e-01"/>
+    <collision name="${prefix}${name}__calf_upper_collision">
+      <origin rpy="0  0  0" xyz="0.09732 0.0 -0.470252"/>
       <geometry>
         <box size="0.397840 0.346075 1.385496"/>
       </geometry>
     </collision>
-    <visual name="${prefix}${name}__visual">
+    <visual name="${prefix}${name}__calf_upper_visual">
       <origin rpy="0  0  0" xyz="0  0  0"/>
       <geometry>
@@ -151,5 +153,5 @@
       <inertia ixx="0.028" ixy="0." ixz="0." iyy="0.022" iyz="0" izz="0.009"/>
     </inertial>
-    <collision name="${prefix}${name}__collision">
+    <collision name="${prefix}${name}__linkage_upper_collision">
       <origin rpy="0  0  0" xyz="1.01380000e-01   0.00000000e+00  -1.00000000e-05"/>
       <geometry>
@@ -157,5 +159,5 @@
       </geometry>
     </collision>
-    <visual name="${prefix}${name}__visual">
+    <visual name="${prefix}${name}__linkage_upper_visual">
       <origin rpy="0  0  0" xyz="0  0  0"/>
       <geometry>
@@ -170,5 +172,5 @@
       <inertia ixx="0.028" ixy="0." ixz="0." iyy="0.022" iyz="0" izz="0.009"/>
     </inertial>
-    <collision name="${prefix}${name}__collision">
+    <collision name="${prefix}${name}__linkage_lower_collision">
       <origin rpy="0  0  0" xyz="1.01380000e-01   0.00000000e+00  -1.00000000e-05"/>
       <geometry>
@@ -176,5 +178,5 @@
       </geometry>
     </collision>
-    <visual name="${prefix}${name}__visual">
+    <visual name="${prefix}${name}__linkage_lower_visual">
       <origin rpy="0  0  0" xyz="0  0  0"/>
       <geometry>
@@ -187,16 +189,15 @@
     <inertial>
       <mass value="18.983"/>
-      <origin rpy="0  0  0" xyz="0.01114  0      -0.10264"/>
+      <origin rpy="0  0  0" xyz="0.048200 0.000000 -0.405153"/>
       <inertia ixx="1.827" ixy="0." ixz="0.243" iyy="1.859" iyz="0." izz="0.145"/>
     </inertial>
-    <collision name="${prefix}${name}__collision">
-      <!--TODO figure out if this position is with a compressed shock -->
-      <origin rpy="0  0  0" xyz="0.01567  0      -0.10663"/>
+    <collision name="${prefix}${name}__calf_lower_collision">
+        <origin rpy="0  0  0" xyz="0.058576 0.000000 -0.4418265"/>
       <geometry>
         <box size="0.237352 0.180975 1.122347"/>
       </geometry>
     </collision>
-    <visual name="${prefix}${name}__visual">
-      <origin rpy="0  0  0" xyz="-0.0371  0      0.3024"/>
+    <visual name="${prefix}${name}__calf_lower_visual">
+      <origin rpy="0  0  0" xyz="0  0  0"/>
       <geometry>
           <mesh filename="package://stompy_description/meshes/calf_lower.stl" scale="1.0 1.0 1.0"/>
@@ -210,11 +211,11 @@
       <inertia ixx="0.002" ixy="0" ixz="0" iyy="0.001" iyz="0" izz="0.002"/>
     </inertial>
-    <collision name="${prefix}${name}__collision">
-      <origin rpy="0  0  0" xyz="0       0      -0.01709"/>
+    <collision name="${prefix}${name}__ankle_collision">
+      <origin rpy="0  0  0" xyz="0       0      -0.019693"/>
       <geometry>
         <box size="0.073025 0.127000 0.100314"/>
       </geometry>
     </collision>
-    <visual name="${prefix}${name}__visual">
+    <visual name="${prefix}${name}__ankle_visual">
       <origin rpy="0  0  0" xyz="0  0  0"/>
       <geometry>
@@ -226,14 +227,14 @@
     <inertial>
       <mass value="9.307"/>
-      <origin rpy="0  0  0" xyz="0       0      -0.11187"/>
+      <origin rpy="0 0 0" xyz="0.000000 0.000000 -0.114469"/>
       <inertia ixx="0.069" ixy="0" ixz="0" iyy="0.069" iyz="0" izz="0.102"/>
     </inertial>
-    <collision name="${prefix}${name}__collision">
-      <origin rpy="0  0  0" xyz="0       0      -0.11187"/>
+    <collision name="${prefix}${name}__foot_collision">
+      <origin rpy="0  0  0" xyz="0       0      -0.05495"/>
       <geometry>
         <box size="0.355474 0.355348 0.188913"/>
       </geometry>
     </collision>
-    <visual name="${prefix}${name}__visual">
+    <visual name="${prefix}${name}__foot_visual">
       <origin rpy="0  0  0" xyz="0  0  0"/>
       <geometry>
@@ -242,4 +243,30 @@
     </visual>
   </link>
+  <link name="${prefix}${name}__pad">
+    <inertial>
+      <mass value="1"/>
+      <origin rpy="0 0 0" xyz="0 0 -0.00635"/>
+      <inertia ixx="0.00348" ixy="0" ixz="0" iyy="0.00348" iyz="0" izz="0.00694"/>
+    </inertial>
+    <collision name="{$prefix}${name}__pad_collision">
+      <origin rpy="0 0 0" xyz="0 0 -0.00635"/>
+      <geometry>
+        <cylinder length="0.0127" radius="0.1778"/>
+      </geometry>
+    </collision>
+    <visual name="${prefix}${name}__pad_visual">
+      <origin rpy="0 0 0" xyz="0 0 -0.00635"/>
+      <geometry>
+        <cylinder length="0.0127" radius="0.1778"/>
+      </geometry>
+    </visual>
+  </link>
+  <gazebo reference="${prefix}${name}__pad">
+    <mu1>15000000000</mu1>
+    <mu2>15000000000</mu2>
+    <fdir1>0 0 0</fdir1>
+    <minDepth>0.0001</minDepth>
+    <maxVel>100000.0</maxVel>
+  </gazebo>
   <joint name="${prefix}body_to_${name}" type="revolute">
     <parent link="${prefix}body"/>
