Commit message: renaming joints

File: src/stompy_description/urdf/stompy.urdf.xacro (robot description, xacro)
@@ -7,11 +7,11 @@
  </gazebo>
  <xacro:include filename="$(find stompy_description)/urdf/stompyleg_macro.urdf.xacro" />
- <link name="stompy__base" />
- <joint name="stompy__base_to_body" type="fixed">
+ <link name="base_link" />
+ <joint name="body" type="fixed">
   <origin xyz="0 0 0" rpy="0 0 0"/>
-  <parent link="stompy__base" />
-  <child link="stompy__body" />
+  <parent link="base_link" />
+  <child link="body_link" />
  </joint>
- <link name="stompy__body">
+ <link name="body_link">
     <inertial>
       <mass value="1823.41"/>
@@ -20,5 +20,5 @@
       <inertia ixx="499.7" ixy="0.019" ixz="-172.0" iyy="3253.0" iyz="0.019" izz="3049.0"/>
     </inertial>
-    <collision name="stompy__collision">
+    <collision name="body_link_collision">
       <origin rpy="0  0  0" xyz="0     0     0"/>
       <geometry>
@@ -26,5 +26,5 @@
       </geometry>
     </collision>
-    <visual name="stompy__visual">
+    <visual name="body_link_visual">
       <origin rpy="0  0  0" xyz="0  0  0"/>
       <geometry>
@@ -33,9 +33,9 @@
     </visual>
   </link>
-  <xacro:leg prefix="stompy__" name="fl" rpy="0 0 0.9599" xyz="2.35117  0.5842   -0.0967"/>
-  <xacro:leg prefix="stompy__" name="fr" rpy="0      0     -0.9599" xyz="2.35117 -0.5842   -0.0967"/>
-  <xacro:leg prefix="stompy__" name="ml" rpy="0      0      1.5706" xyz="0.0  0.6858   -0.0967"/>
-  <xacro:leg prefix="stompy__" name="mr" rpy="0      0     -1.5706" xyz="0.0 -0.6858   -0.0967"/>
-  <xacro:leg prefix="stompy__" name="rl" rpy="0      0      2.1816" xyz="-2.35117  0.5842  -0.0967"/>
-  <xacro:leg prefix="stompy__" name="rr" rpy="0      0     -2.1816" xyz="-2.35117 -0.5842  -0.0967"/>
+  <xacro:leg name="fl" rpy="0 0 0.9599" xyz="2.35117  0.5842   -0.0967"/>
+  <xacro:leg name="fr" rpy="0 0 -0.9599" xyz="2.35117 -0.5842   -0.0967"/>
+  <xacro:leg name="ml" rpy="0 0 1.5706" xyz="0.0  0.6858   -0.0967"/>
+  <xacro:leg name="mr" rpy="0 0 -1.5706" xyz="0.0 -0.6858   -0.0967"/>
+  <xacro:leg name="rl" rpy="0 0 2.1816" xyz="-2.35117  0.5842  -0.0967"/>
+  <xacro:leg name="rr" rpy="0 0 -2.1816" xyz="-2.35117 -0.5842  -0.0967"/>
 </robot>

File: src/stompy_description/urdf/stompyleg_macro.urdf.xacro (robot description, xacro)
@@ -3,8 +3,7 @@
  <xacro:property name="max_e" value="10000000"/>
  <xacro:property name="max_v" value="10"/>
- <xacro:macro name="leg" params="prefix name rpy xyz">
-  <joint name="${prefix}${name}__hip_to_thigh" type="revolute">
-    <parent link="${prefix}${name}__hip"/>
-    <child link="${prefix}${name}__thigh"/>
+ <xacro:macro name="leg" params="name rpy xyz"> <joint name="${name}_thigh" type="revolute">
+    <parent link="${name}_hip_link"/>
+    <child link="${name}_thigh_link"/>
     <origin rpy="0  0  0" xyz="0.279  0     0"/>
     <axis xyz="0  1  0"/>
@@ -12,7 +11,7 @@
     <dynamics damping="10000.0" />
   </joint>
-  <joint name="${prefix}${name}__thigh_to_calf_upper" type="revolute">
-    <parent link="${prefix}${name}__thigh"/>
-    <child link="${prefix}${name}__calf_upper"/>
+  <joint name="${name}_knee" type="revolute">
+    <parent link="${name}_thigh_link"/>
+    <child link="${name}_calf_upper_link"/>
     <origin rpy="0  0  0" xyz="0.143  0       1.364"/>
     <axis xyz="0  1  0"/>
@@ -22,7 +21,7 @@
   </joint>
   <!--
-  <joint name="${prefix}${name}__calf_upper_to_linkage_upper" type="fixed">
-    <parent link="${prefix}${name}__calf_upper"/>
-    <child link="${prefix}${name}__linkage_upper"/>
+  <joint name="${name}__calf_upper_to_linkage_upper" type="fixed">
+    <parent link="${name}__calf_upper"/>
+    <child link="${name}__linkage_upper"/>
     <origin rpy="0  0  0" xyz="0.0016  0     -0.8185"/>
     <axis xyz="0  1  0"/>
@@ -30,7 +29,7 @@
     <dynamics damping="10000.0" />
   </joint>
-  <joint name="${prefix}${name}__calf_upper_to_linkage_lower" type="fixed">
-    <parent link="${prefix}${name}__calf_upper"/>
-    <child link="${prefix}${name}__linkage_lower"/>
+  <joint name="${name}__calf_upper_to_linkage_lower" type="fixed">
+    <parent link="${name}__calf_upper"/>
+    <child link="${name}__linkage_lower"/>
     <origin rpy="0  0  0" xyz="0.0388  0     -1.121"/>
     <axis xyz="0  1  0"/>
@@ -39,7 +38,7 @@
   </joint>
   -->
-  <joint name="${prefix}${name}__calf_upper_to_calf_lower" type="prismatic">
-    <parent link="${prefix}${name}__calf_upper"/>
-    <child link="${prefix}${name}__calf_lower"/>
+  <joint name="${name}_calf" type="prismatic">
+    <parent link="${name}_calf_upper_link"/>
+    <child link="${name}_calf_lower_link"/>
     <origin rpy="0  0  0" xyz="0.203  0   -0.847"/>
     <axis xyz="0  0  1"/>
@@ -48,14 +47,14 @@
   </joint>
   <!--
-  <joint name="${prefix}${name}__linkage_upper_to_calf_lower" type="revolute">
-    <parent link="${prefix}${name}__linkage_upper"/>
-    <child link="${prefix}${name}__calf_lower"/>
+  <joint name="${name}__linkage_upper_to_calf_lower" type="revolute">
+    <parent link="${name}__linkage_upper"/>
+    <child link="${name}__calf_lower"/>
     <origin rpy="0  0  0" xyz="0.203  0     0"/>
     <axis xyz="0  1  0"/>
     <limit effort="${max_e}" lower="0.0" upper="0.349" velocity="${max_v}"/>
   </joint>
-  <joint name="${prefix}${name}__linkage_lower_to_calf_lower" type="fixed">
-    <parent link="${prefix}${name}__linkage_lower"/>
-    <child link="${prefix}${name}__calf_lower"/>
+  <joint name="${name}__linkage_lower_to_calf_lower" type="fixed">
+    <parent link="${name}__linkage_lower"/>
+    <child link="${name}__calf_lower"/>
     <origin rpy="0  0  0" xyz="2.02900000e-01   0.00000000e+00   1.00000000e-04"/>
     <axis xyz="0  1  0"/>
@@ -63,7 +62,7 @@
   </joint>
   -->
-  <joint name="${prefix}${name}__calf_lower_to_ankle" type="revolute">
-    <parent link="${prefix}${name}__calf_lower"/>
-    <child link="${prefix}${name}__ankle"/>
+  <joint name="${name}_ankle" type="revolute">
+    <parent link="${name}_calf_lower_link"/>
+    <child link="${name}_ankle_link"/>
     <origin rpy="0  0  0" xyz="0.02  0     -0.968"/>
     <axis xyz="0  1  0"/>
@@ -71,7 +70,7 @@
     <dynamics damping="1.0" />
   </joint>
-  <joint name="${prefix}${name}__ankle_to_foot" type="revolute">
-    <parent link="${prefix}${name}__ankle"/>
-    <child link="${prefix}${name}__foot"/>
+  <joint name="${name}_foot" type="revolute">
+    <parent link="${name}_ankle_link"/>
+    <child link="${name}_foot_link"/>
     <origin rpy="0  0  0" xyz="0      0     -0.0412"/>
     <axis xyz="1  0  0"/>
@@ -79,11 +78,11 @@
     <dynamics damping="1.0" />
 </joint>
-  <joint name="${prefix}${name}__foot_to_pad" type="continuous">
-    <parent link="${prefix}${name}__foot"/>
-    <child link="${prefix}${name}__pad"/>
+  <joint name="${name}_pad" type="continuous">
+    <parent link="${name}_foot_link"/>
+    <child link="${name}_pad_link"/>
     <origin rpy="0 0 0" xyz="0 0 -0.153"/>
     <axis xyz="0 0 1"/>
   </joint>
-  <link name="${prefix}${name}__hip">
+  <link name="${name}_hip_link">
     <inertial>
       <mass value="28.231"/>
@@ -91,5 +90,5 @@
       <inertia ixx="0.417" ixy="0." ixz="0.026" iyy="0.327" iyz="0." izz="0.337"/>
     </inertial>
-    <collision name="${prefix}${name}__hip_collision">
+    <collision name="${name}_hip_link_collision">
       <origin rpy="0  0  0" xyz="0.1341685 -0.000000 0.096707"/>
       <geometry>
@@ -97,5 +96,5 @@
       </geometry>
     </collision>
-    <visual name="${prefix}${name}__hip_visual">
+    <visual name="${name}_hip_link_visual">
       <origin rpy="0  0  0" xyz="0  0  0"/>
       <geometry>
@@ -104,5 +103,5 @@
     </visual>
   </link>
-  <link name="${prefix}${name}__thigh">
+  <link name="${name}_thigh_link">
     <inertial>
       <mass value="64.053"/>
@@ -110,5 +109,5 @@
       <inertia ixx="10.62" ixy="0." ixz="-0.34" iyy="10.92" iyz="0." izz="1.334"/>
     </inertial>
-    <collision name="${prefix}${name}__thigh_collision">
+    <collision name="${name}_thigh_link_collision">
       <origin rpy="0  0  0" xyz="-0.078093 -0.000000 0.6820835"/>
       <geometry>
@@ -116,5 +115,5 @@
       </geometry>
     </collision>
-    <visual name="${prefix}${name}__thigh_visual">
+    <visual name="${name}_thigh_link_visual">
       <origin rpy="0  0  0" xyz="0  0  0"/>
       <geometry>
@@ -123,5 +122,5 @@
     </visual>
   </link>
-  <link name="${prefix}${name}__calf_upper">
+  <link name="${name}_calf_upper_link">
     <inertial>
       <mass value="39.145"/>
@@ -129,5 +128,5 @@
       <inertia ixx="5.471" ixy="0." ixz="1.148" iyy="5.636" iyz="0." izz="0.775"/>
     </inertial>
-    <collision name="${prefix}${name}__calf_upper_collision">
+    <collision name="${name}_calf_upper_link_collision">
       <origin rpy="0  0  0" xyz="0.09732 0.0 -0.470252"/>
       <geometry>
@@ -135,5 +134,5 @@
       </geometry>
     </collision>
-    <visual name="${prefix}${name}__calf_upper_visual">
+    <visual name="${name}_calf_upper_link_visual">
       <origin rpy="0  0  0" xyz="0  0  0"/>
       <geometry>
@@ -143,5 +142,5 @@
   </link>
   <!--
-  <link name="${prefix}${name}__linkage_upper">
+  <link name="${name}__linkage_upper">
     <inertial>
       <mass value="3.754"/>
@@ -149,5 +148,5 @@
       <inertia ixx="0.028" ixy="0." ixz="0." iyy="0.022" iyz="0" izz="0.009"/>
     </inertial>
-    <collision name="${prefix}${name}__linkage_upper_collision">
+    <collision name="${name}__linkage_upper_collision">
       <origin rpy="0  0  0" xyz="1.01380000e-01   0.00000000e+00  -1.00000000e-05"/>
       <geometry>
@@ -155,5 +154,5 @@
       </geometry>
     </collision>
-    <visual name="${prefix}${name}__linkage_upper_visual">
+    <visual name="${name}__linkage_upper_visual">
       <origin rpy="0  0  0" xyz="0  0  0"/>
       <geometry>
@@ -162,5 +161,5 @@
     </visual>
   </link>
-  <link name="${prefix}${name}__linkage_lower">
+  <link name="${name}__linkage_lower">
     <inertial>
       <mass value="3.754"/>
@@ -168,5 +167,5 @@
       <inertia ixx="0.028" ixy="0." ixz="0." iyy="0.022" iyz="0" izz="0.009"/>
     </inertial>
-    <collision name="${prefix}${name}__linkage_lower_collision">
+    <collision name="${name}__linkage_lower_collision">
       <origin rpy="0  0  0" xyz="1.01380000e-01   0.00000000e+00  -1.00000000e-05"/>
       <geometry>
@@ -174,5 +173,5 @@
       </geometry>
     </collision>
-    <visual name="${prefix}${name}__linkage_lower_visual">
+    <visual name="${name}__linkage_lower_visual">
       <origin rpy="0  0  0" xyz="0  0  0"/>
       <geometry>
@@ -182,5 +181,5 @@
   </link>
   -->
-  <link name="${prefix}${name}__calf_lower">
+  <link name="${name}_calf_lower_link">
     <inertial>
       <mass value="18.983"/>
@@ -188,5 +187,5 @@
       <inertia ixx="1.827" ixy="0." ixz="0.243" iyy="1.859" iyz="0." izz="0.145"/>
     </inertial>
-    <collision name="${prefix}${name}__calf_lower_collision">
+    <collision name="${name}_calf_lower_link_collision">
         <origin rpy="0  0  0" xyz="0.058576 0.000000 -0.4418265"/>
       <geometry>
@@ -194,5 +193,5 @@
       </geometry>
     </collision>
-    <visual name="${prefix}${name}__calf_lower_visual">
+    <visual name="${name}_calf_lower_link_visual">
       <origin rpy="0  0  0" xyz="0  0  0"/>
       <geometry>
@@ -201,5 +200,5 @@
     </visual>
   </link>
-  <link name="${prefix}${name}__ankle">
+  <link name="${name}_ankle_link">
     <inertial>
       <mass value="1.391"/>
@@ -207,5 +206,5 @@
       <inertia ixx="0.002" ixy="0" ixz="0" iyy="0.001" iyz="0" izz="0.002"/>
     </inertial>
-    <collision name="${prefix}${name}__ankle_collision">
+    <collision name="${name}_ankle_link_collision">
       <origin rpy="0  0  0" xyz="0       0      -0.019693"/>
       <geometry>
@@ -213,5 +212,5 @@
       </geometry>
     </collision>
-    <visual name="${prefix}${name}__ankle_visual">
+    <visual name="${name}_ankle_link_visual">
       <origin rpy="0  0  0" xyz="0  0  0"/>
       <geometry>
@@ -220,5 +219,5 @@
     </visual>
   </link>
-  <link name="${prefix}${name}__foot">
+  <link name="${name}_foot_link">
     <inertial>
       <mass value="9.307"/>
@@ -226,5 +225,5 @@
       <inertia ixx="0.069" ixy="0" ixz="0" iyy="0.069" iyz="0" izz="0.102"/>
     </inertial>
-    <collision name="${prefix}${name}__foot_collision">
+    <collision name="${name}_foot_link_collision">
       <origin rpy="0  0  0" xyz="0       0      -0.05495"/>
       <geometry>
@@ -232,5 +231,5 @@
       </geometry>
     </collision>
-    <visual name="${prefix}${name}__foot_visual">
+    <visual name="${name}_foot_link_visual">
       <origin rpy="0  0  0" xyz="0  0  0"/>
       <geometry>
@@ -239,5 +238,5 @@
     </visual>
 </link>
-  <gazebo reference="${prefix}${name}__foot">
+  <gazebo reference="${name}_foot_link">
     <mu1>50</mu1>
     <mu2>50</mu2>
@@ -245,5 +244,5 @@
     <minDepth>0.0000003</minDepth>
   </gazebo>
-  <link name="${prefix}${name}__pad">
+  <link name="${name}_pad_link">
     <inertial>
       <mass value="1"/>
@@ -251,5 +250,5 @@
       <inertia ixx="0.00348" ixy="0" ixz="0" iyy="0.00348" iyz="0" izz="0.00694"/>
     </inertial>
-    <collision name="{$prefix}${name}__pad_collision">
+    <collision name="{$prefix}${name}_pad_link_collision">
       <origin rpy="0 0 0" xyz="0 0 -0.00635"/>
       <geometry>
@@ -257,5 +256,5 @@
       </geometry>
     </collision>
-    <visual name="${prefix}${name}__pad_visual">
+    <visual name="${name}__pad_link_visual">
       <origin rpy="0 0 0" xyz="0 0 -0.00635"/>
       <geometry>
@@ -264,5 +263,5 @@
     </visual>
   </link>
-  <gazebo reference="${prefix}${name}__pad">
+  <gazebo reference="${name}_pad_link">
     <mu1>500</mu1>
     <mu2>500</mu2>
@@ -270,7 +269,7 @@
     <minDepth>0.0000003</minDepth>
   </gazebo>
-  <joint name="${prefix}body_to_${name}" type="revolute">
-    <parent link="${prefix}body"/>
-    <child link="${prefix}${name}__hip"/>
+  <joint name="${name}_hip" type="revolute">
+    <parent link="body_link"/>
+    <child link="${name}_hip_link"/>
     <origin rpy="${rpy}" xyz="${xyz}"/>
     <axis xyz="0  0  1"/>
@@ -279,40 +278,40 @@
   </joint>
   <!-- transmission added for gazebo_ros_control, needed for every joint -->
-  <transmission name="${prefix}body_to_${name}_tran">
+  <transmission name="${name}_hip_tran">
     <type>transmission_interface/SimpleTransmission</type>
-    <joint name="${prefix}body_to_${name}">
+    <joint name="${name}_hip">
       <hardwareInterface>EffortJointInterface</hardwareInterface>
     </joint>
-    <actuator name="${prefix}body_to_${name}_motor">
+    <actuator name="${name}_hip_motor">
       <hardwareInterface>EffortJointInterface</hardwareInterface>
       <mechanicalReduction>1</mechanicalReduction>
     </actuator>
   </transmission>
-  <transmission name="${prefix}${name}_hip_to_thigh_tran">
+  <transmission name="${name}_thigh_tran">
     <type>transmission_interface/SimpleTransmission</type>
-    <joint name="${prefix}${name}__hip_to_thigh">
+    <joint name="${name}_thigh">
       <hardwareInterface>EffortJointInterface</hardwareInterface>
     </joint>
-    <actuator name="${prefix}${name}_hip_to_thigh_motor">
+    <actuator name="${name}_thigh_motor">
       <hardwareInterface>EffortJointInterface</hardwareInterface>
       <mechanicalReduction>1</mechanicalReduction>
     </actuator>
   </transmission>
-  <transmission name="${prefix}${name}_thigh_to_calf_upper_tran">
+  <transmission name="${name}_knee_tran">
     <type>transmission_interface/SimpleTransmission</type>
-    <joint name="${prefix}${name}__thigh_to_calf_upper">
+    <joint name="${name}_knee">
       <hardwareInterface>EffortJointInterface</hardwareInterface>
     </joint>
-    <actuator name="${prefix}${name}_thigh_to_calf_upper_motor">
+    <actuator name="${name}_knee_motor">
       <hardwareInterface>EffortJointInterface</hardwareInterface>
       <mechanicalReduction>1</mechanicalReduction>
     </actuator>
   </transmission>
-  <transmission name="${prefix}${name}_calf_upper_to_calf_lower_tran">
+  <transmission name="${name}_calf_tran">
     <type>transmission_interface/SimpleTransmission</type>
-    <joint name="${prefix}${name}__calf_upper_to_calf_lower">
+    <joint name="${name}_calf">
       <hardwareInterface>EffortJointInterface</hardwareInterface>
     </joint>
-    <actuator name="${prefix}${name}_calf_upper_to_calf_lower_motor">
+    <actuator name="${name}_calf_motor">
       <hardwareInterface>EffortJointInterface</hardwareInterface>
       <mechanicalReduction>1</mechanicalReduction>

Commit message: adding driver camera

File: src/stompy_description/urdf/stompy.urdf.xacro (robot description, xacro)
@@ -41,4 +41,74 @@
     </visual>
   </link>
+  <gazebo reference="camera_link">
+    <material>Gazebo/Red</material>
+  </gazebo>
+  <joint name="camera_joint" type="fixed">
+    <axis xyz="0 1 0" />
+    <origin xyz="1.5 0.25 0.75" rpy="0 0 0"/>
+    <parent link="body_link"/>
+    <child link="camera_link"/>
+  </joint>
+  <link name="camera_link">
+    <collision>
+      <origin xyz="0 0 0" rpy="0 0 0"/>
+      <geometry>
+    <box size="0.05 0.05 0.05"/>
+      </geometry>
+    </collision>
+    <visual>
+      <origin xyz="0 0 0" rpy="0 0 0"/>
+      <geometry>
+        <box size="0.05 0.05 0.05"/>
+      </geometry>
+      <material name="red">
+        <color rgba="1.0 0. 0. 1.0"/>
+      </material>
+    </visual>
+    <inertial>
+      <mass value="1e-5" />
+      <origin xyz="0 0 0" rpy="0 0 0"/>
+      <inertia ixx="1e-6" ixy="0" ixz="0" iyy="1e-6" iyz="0" izz="1e-6" />
+    </inertial>
+  </link>
+ <gazebo reference="camera_link">
+    <sensor type="camera" name="camera1">
+      <update_rate>30.0</update_rate>
+      <camera name="head">
+        <horizontal_fov>1.3962634</horizontal_fov>
+        <image>
+          <width>800</width>
+          <height>800</height>
+          <format>R8G8B8</format>
+        </image>
+        <clip>
+          <near>0.02</near>
+          <far>300</far>
+        </clip>
+        <noise>
+          <type>gaussian</type>
+          <!-- Noise is sampled independently per pixel on each frame.
+               That pixel's noise value is added to each of its color
+               channels, which at that point lie in the range [0,1]. -->
+          <mean>0.0</mean>
+          <stddev>0.007</stddev>
+        </noise>
+      </camera>
+      <plugin name="camera_controller" filename="libgazebo_ros_camera.so">
+        <alwaysOn>true</alwaysOn>
+        <updateRate>0.0</updateRate>
+        <cameraName>rrbot/camera1</cameraName>
+        <imageTopicName>image_raw</imageTopicName>
+        <cameraInfoTopicName>camera_info</cameraInfoTopicName>
+        <frameName>camera_link</frameName>
+        <hackBaseline>0.07</hackBaseline>
+        <distortionK1>0.0</distortionK1>
+        <distortionK2>0.0</distortionK2>
+        <distortionK3>0.0</distortionK3>
+        <distortionT1>0.0</distortionT1>
+        <distortionT2>0.0</distortionT2>
+      </plugin>
+    </sensor>
+  </gazebo>
   <xacro:leg name="fl" rpy="0 0 0.9599" xyz="2.2352  0.5842   -0.1000"/>
   <xacro:leg name="fr" rpy="0 0 -0.9599" xyz="2.2352 -0.5842   -0.1000"/>
